Commit message: walkerbro deleted

File: mors/urdf/mors_for_nav.urdf (robot description, URDF)
Before this commit: robot walkerbro, 21 links, 20 joints
Links:
- link abad_L1: geometry collision mesh filename=package://mors/urdf/meshes_for_nav/joint1.stl scale=1 1 1; visual mesh filename=package://mors/urdf/meshes_for_nav/joint1.stl scale=1 1 1
- link abad_L2: geometry collision mesh filename=package://mors/urdf/meshes_for_nav/joint1.stl scale=1 1 1; visual mesh filename=package://mors/urdf/meshes_for_nav/joint1.stl scale=1 1 1
- link abad_R1: geometry collision mesh filename=package://mors/urdf/meshes_for_nav/joint1.stl scale=1 1 1; visual mesh filename=package://mors/urdf/meshes_for_nav/joint1.stl scale=1 1 1
- link abad_R2: geometry collision mesh filename=package://mors/urdf/meshes_for_nav/joint1.stl scale=1 1 1; visual mesh filename=package://mors/urdf/meshes_for_nav/joint1.stl scale=1 1 1
- link base_link: geometry collision mesh filename=package://mors/urdf/meshes_for_nav/body.stl scale=1 1 1; visual mesh filename=package://mors/urdf/meshes_for_nav/body.stl scale=1 1 1
- link hip_L1: geometry collision mesh filename=package://mors/urdf/meshes_for_nav/joint2.stl scale=1 1 1; visual mesh filename=package://mors/urdf/meshes_for_nav/joint2.stl scale=1 1 1
- link hip_L2: geometry collision mesh filename=package://mors/urdf/meshes_for_nav/joint2.stl scale=1 1 1; visual mesh filename=package://mors/urdf/meshes_for_nav/joint2.stl scale=1 1 1
- link hip_R1: geometry collision mesh filename=package://mors/urdf/meshes_for_nav/joint2.stl scale=1 1 1; visual mesh filename=package://mors/urdf/meshes_for_nav/joint2.stl scale=1 1 1
- link hip_R2: geometry collision mesh filename=package://mors/urdf/meshes_for_nav/joint2.stl scale=1 1 1; visual mesh filename=package://mors/urdf/meshes_for_nav/joint2.stl scale=1 1 1
- link knee_L1: geometry collision mesh filename=package://mors/urdf/meshes_for_nav/joint3.stl scale=1 1 1; visual mesh filename=package://mors/urdf/meshes_for_nav/joint3.stl scale=1 1 1
- link knee_L2: geometry collision mesh filename=package://mors/urdf/meshes_for_nav/joint3.stl scale=1 1 1; visual mesh filename=package://mors/urdf/meshes_for_nav/joint3.stl scale=1 1 1
- link knee_R1: geometry collision mesh filename=package://mors/urdf/meshes_for_nav/joint3.stl scale=1 1 1; visual mesh filename=package://mors/urdf/meshes_for_nav/joint3.stl scale=1 1 1
- link knee_R2: geometry collision mesh filename=package://mors/urdf/meshes_for_nav/joint3.stl scale=1 1 1; visual mesh filename=package://mors/urdf/meshes_for_nav/joint3.stl scale=1 1 1
- link scan_frame: geometry collision box size=0.058 0.058 0.087; visual mesh filename=package://mors/urdf/meshes_for_nav/rplidar_a1.stl
